File: starter_board.kicad_pcb (KiCad board)
At the start: 2 copper layers, 102 x 40 mm, 44 parts, among them J1 Conn_01x10, J2 Conn_01x10, J3 ICSP, J4 USB_B_Micro, SW1 SW_Push, U1 ATmega32U4-A, Y1 16MHz

Commit message: Add files via upload
Edit #1
Parts:
- moved SW1 3.35 mm to (88.0, 158.3), turned to -90 degrees
Routing:
- net /D7: track 41.6 -> 30.8 mm
- net GND: track 8.72 -> 0.00 mm
Changed lines of the file:
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@@
 	(footprint "Button_Switch_SMD:SW_SPST_PTS647_Sx38"
 		(layer "F.Cu")
-		(at 91.006 156.792)
+		(at 88.006 158.292 -90)
 		(descr "C&K Components SPST SMD PTS647 Series 4.5mm Tact Switch, 3.8mm Height, see https://www.ckswitches.com/media/2567/pts647.pdf")
 		(tags "SPST Button Switch")
 		(property "Reference" "SW1"
-			(at 0 -4.05 0)
+			(at 0 -4.05 90)
 			(layer "F.SilkS")
 			(effects
@@
 		)
 		(property "Value" "SW_Push"
-			(at 0 4.15 0)
+			(at 0 4.15 90)
 			(layer "F.Fab")
 			(effects
@@
 		)
 		(property "Footprint" "Button_Switch_SMD:SW_SPST_PTS647_Sx38"
-			(at 0 0 0)
+			(at 0 0 -90)
 			(unlocked yes)
 			(layer "F.Fab")
@@
 		)
 		(property "Datasheet" ""
-			(at 0 0 0)
+			(at 0 0 -90)
 			(unlocked yes)
 			(layer "F.Fab")
@@
 		)
 		(property "Description" "Push button switch, generic, two pins"
-			(at 0 5.7 0)
+			(at 0 5.7 -90)
 			(unlocked yes)
 			(layer "F.Fab")
@@
 		(attr smd)
 		(fp_line
-			(start -2.45 -2.45)
-			(end -2.45 -2.4)
+			(start -2.45 2.45)
+			(end 2.45 2.45)
 			(stroke
 				(width 0.12)
@@
 		)
 		(fp_line
-			(start -2.45 -2.45)
-			(end 2.45 -2.45)
+			(start -2.45 2.45)
+			(end -2.45 2.4)
 			(stroke
 				(width 0.12)
@@
 		)
 		(fp_line
-			(start -2.45 -0.75)
-			(end -2.45 0.75)
+			(start 2.45 2.45)
+			(end 2.45 2.4)
 			(stroke
 				(width 0.12)
@@
 		)
 		(fp_line
-			(start -2.45 2.45)
-			(end -2.45 2.4)
+			(start -2.45 -0.75)
+			(end -2.45 0.75)
 			(stroke
 				(width 0.12)
@@
 		)
 		(fp_line
-			(start -2.45 2.45)
-			(end 2.45 2.45)
+			(start 2.45 -0.75)
+			(end 2.45 0.75)
 			(stroke
 				(width 0.12)
@@
 		)
 		(fp_line
-			(start 2.45 -2.45)
-			(end 2.45 -2.4)
+			(start -2.45 -2.45)
+			(end -2.45 -2.4)
 			(stroke
 				(width 0.12)
@@
 		)
 		(fp_line
-			(start 2.45 -0.75)
-			(end 2.45 0.75)
+			(start -2.45 -2.45)
+			(end 2.45 -2.45)
 			(stroke
 				(width 0.12)
@@
 		)
 		(fp_line
-			(start 2.45 2.45)
-			(end 2.45 2.4)
+			(start 2.45 -2.45)
+			(end 2.45 -2.4)
 			(stroke
 				(width 0.12)
@@
 		)
 		(fp_text user "${REFERENCE}"
-			(at 0 -4.05 0)
+			(at 0 -4.05 90)
 			(layer "F.Fab")
 			(effects
@@
 		)
 		(pad "1" smd roundrect
-			(at -2.625 -1.6)
+			(at -2.625 -1.6 270)
 			(size 1.55 1)
 			(layers "F.Cu" "F.Paste" "F.Mask")
@@
 		)
 		(pad "1" smd roundrect
-			(at 2.625 -1.6)
+			(at 2.625 -1.6 270)
 			(size 1.55 1)
 			(layers "F.Cu" "F.Paste" "F.Mask")
@@
 		)
 		(pad "2" smd roundrect
-			(at -2.625 1.6)
+			(at -2.625 1.6 270)
 			(size 1.55 1)
 			(layers "F.Cu" "F.Paste" "F.Mask")
@@
 		)
 		(pad "2" smd roundrect
-			(at 2.625 1.6)
+			(at 2.625 1.6 270)
 			(size 1.55 1)
 			(layers "F.Cu" "F.Paste" "F.Mask")
@@
 	)
 	(segment
-		(start 94.756 157.717)
-		(end 94.756 155.592)
-		(width 0.25)
-		(layer "F.Cu")
-		(net 2)
-	)
-	(segment
-		(start 94.506 157.967)
-		(end 93.9859 157.967)
-		(width 0.25)
-		(layer "F.Cu")
-		(net 2)
-	)
-	(segment
-		(start 94.506 157.967)
-		(end 94.756 157.717)
-		(width 0.25)
-		(layer "F.Cu")
-		(net 2)
-	)
-	(segment
-		(start 94.756 155.592)
-		(end 89.506 155.592)
-		(width 0.25)
-		(layer "F.Cu")
-		(net 2)
-	)
-	(segment
-		(start 93.9859 157.967)
-		(end 93.656 158.2969)
-		(width 0.25)
-		(layer "F.Cu")
-		(net 2)
-	)
-	(segment
 		(start 69.414 155.9895)
 		(end 69.342 156.0615)
@@
 	)
 	(segment
-		(start 89.506 158.792)
-		(end 84.537 158.792)
-		(width 0.25)
-		(layer "F.Cu")
-		(net 68)
-	)
-	(segment
 		(start 63.26 138.24)
 		(end 62.26 138.24)
@@
 	)
 	(segment
-		(start 94.506 159.042)
-		(end 94.506 159.292)
-		(width 0.25)
-		(layer "F.Cu")
-		(net 68)
-	)
-	(segment
-		(start 94.506 159.042)
-		(end 94.756 158.792)
-		(width 0.25)
-		(layer "F.Cu")
-		(net 68)
-	)
-	(segment
 		(start 63.909 138.889)
 		(end 63.26 138.24)
 		(width 0.25)
 		(layer "F.Cu")
-		(net 68)
-	)
-	(segment
-		(start 94.756 158.792)
-		(end 89.506 158.792)
-		(width 0.25)
-		(layer "F.Cu")
